Commit message: homework 3 done

File: urdf/sensors/oakd.urdf.xacro (robot description, xacro)
@@ -44,5 +44,5 @@
       <parent link="${base_frame}"/>
       <child link="${name}_rgb_camera_frame"/>
-      <origin xyz="0 0 0" rpy="0 0 0" />
+      <origin xyz="0 -0.25 0" rpy="0 0 0" />
   </joint>
   <link name="${name}_rgb_camera_optical_frame">
@@ -101,5 +101,5 @@
     <sensor name="rgbd_camera" type="rgbd_camera">
       <camera>
-        <horizontal_fov>1.25</horizontal_fov>
+        <horizontal_fov>1.0</horizontal_fov>
         <image>
           <width>320</width>
@@ -107,5 +107,5 @@
         </image>
         <clip>
-          <near>0.3</near>
+          <near>0.05</near>
           <far>100</far>
         </clip>
